File: schematic/schematic/GatewayV1/GatewayV1.kicad_pcb (KiCad board)
At the start: 2 copper layers, 111 x 111.5 mm, 93 parts, among them J1 0Ω, J2 0Ω, Q4 BSS138, SW1 SW_Push, U10 LMV358, U11 AP63357DV-7, U12 AP63357DV-7, U2 2.4GHz

Commit message: Feat Board Completed, in production
Parts:
- added H1: MountingHole, MountingHole:MountingHole_2.7mm_M2.5, F.Cu at (229.4, 25.6)
- added H2: MountingHole, MountingHole:MountingHole_2.7mm_M2.5, F.Cu at (164.6, 76.0)
- added H3: MountingHole, MountingHole:MountingHole_2.7mm_M2.5, F.Cu at (255.4, 118.6)
- added H4: MountingHole, MountingHole:MountingHole_2.7mm_M2.5, F.Cu at (215.8, 58.4)
- added H5: MountingHole, MountingHole:MountingHole_2.7mm_M2.5, F.Cu at (229.2, 48.2)
- added H6: MountingHole, MountingHole:MountingHole_2.7mm_M2.5, F.Cu at (187.2, 34.2)
- C15: value 47pF -> 33pF
- C4, C5: value C -> 100nF
- D2: value US1MF/1N4007 -> US1MF
- L2: value 6.8uH -> 4.7uH
- P1, P2: value ~ -> CONN-TH-6P-P5.00
- Q1, Q2, Q3: value ~ -> MMBT5401
- Q4: value BSS138 -> BSS138-7-F
- R25, R26, R27, R28: value 22K (FHV) -> R
- R30: value 2kΩ/2.2K -> 2kΩ
- R41: value 220kΩ -> 91kΩ
- R42: value 41.2kΩ -> 30kΩ
- RV1: value R_100K -> 100kΩ
- SW1: value SW_Push -> Btn
- U1, U3: value ~ -> Pin Header 2x6
- U10: value LMV358 -> LMV358IDR
- U13: value ~ -> Red LED
- U2: value 2.4GHz -> ESP8266MOD
- U4: value ~ -> SN74LVC1G08DCKR
- U5: value ~ -> RAK3172-9
- U6: value ~ -> SN74LVC1G32DBVR
- U7: value ~ -> ADS1115IDGSR
- U8: value ~ -> Conn_01x02_Pin
- U9: value ~ -> Opto Peon
- moved C18 1.38 mm to (255.9, 63.1)
- moved C19 1.34 mm to (255.9, 60.2)
- moved C17 0.65 mm to (202.9, 73.8)
- moved U6 0.45 mm to (255.5, 100.1)
Routing:
- net +3.3V: track 308.2 -> 350.8 mm, vias 12 -> 28
- net +5V: track 225.3 -> 264.9 mm, vias 4 -> 18
- net +12V: track 39.4 -> 73.1 mm, vias 0 -> 10
- net GND: track 457.6 -> 486.7 mm, vias 28 -> 67
- net SDA: track 59.5 -> 78.6 mm, vias 2 -> 3
- net SCL: track 70.2 -> 81.1 mm, vias 2 -> 3
- net LORA_RX: track 23.2 -> 32.1 mm, vias 0 -> 1
- net ESP_TX: track 26.3 -> 33.9 mm, vias 1 -> 2
- added copper zone on B.Cu, net +12V
- added copper zone on B.Cu, net +3.3V
- added copper zone on B.Cu, net +5V
