File: schematic/schematic/GatewayV1/peon_voltage_reducer.kicad_sch (KiCad schematic)
At the start: 14 parts, among them Q1 BSS138, Q2 SFH3201, U2 LM358

Commit message: Refactor: Updated ESP
Other:
- note added: "8800v, en vacio. Resolucion de 100v. 5000v aun respeta el animal"
Changed lines of the file:
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@@
 	(generator_version "9.0")
 	(paper "A4")
+	(text "8800v, en vacio.\nResolucion de 100v.\n5000v aun respeta el animal"
+		(exclude_from_sim no)
+		(at 186.182 137.16 0)
+		(effects
+			(font
+				(size 1.27 1.27)
+			)
+		)
+	)
 	(junction
 		(at 204.47 100.33)

Commit message: Feat: Updated components
Parts:
- removed Q2: SFH3201, OptoDevice:Osram_SFH9x0x, symbol Sensor_Optical:SFH3201
- removed U2: LM358, symbol Amplifier_Operational:LM358
- added D2: W10M, easyEDA:DIO-BG-TH_W10M, symbol easyEDA:W10M
- added R12, R13, R14, R17: R, symbol Device:R
- added U2: ~, easyEDA:CONN-TH_KF88SA-16.0-2P, symbol easyEDA:KF88SA-16.0-2P
- added U3: LMV358, easyEDA:SOIC-8_L4.9-W3.9-P1.27-LS6.0-BL, symbol easyEDA:LMV358IDR
- added U7: ~, ibSolutions:PEON_IR_INSULATION_v1, symbol ibSolutions:Peon_IR_High_Voltage_Insulation
- C1: value C -> 100nF; footprint (none) -> easyEDA:C1206; symbol Device:C -> easyEDA:CL31B104KBCNNNC; LCSC Part Name (none) -> 100nF ±10% 50V; Manufacturer (none) -> SAMSUNG(三星); Manufacturer Part (none) -> CL31B104KBCNNNC; Supplier (none) -> LCSC; Supplier Part (none) -> C24497
- C2, C3: footprint (none) -> easyEDA:C1206; symbol Device:C -> easyEDA:CC1206KRX7R9BB104; LCSC Part Name (none) -> 100nF ±10% 50V; Manufacturer (none) -> YAGEO(国巨); Manufacturer Part (none) -> CC1206KRX7R9BB104; Supplier (none) -> LCSC; Supplier Part (none) -> C82601
- D1: value 1N4007 -> US1MF/1N4007; footprint Diode_THT:D_DO-41_SOD81_P10.16mm_Horizontal -> easyEDA:SMAF_L3.5-W2.6-LS4.7-RD; symbol Diode:1N4007 -> easyEDA:US1MF_C64877; LCSC Part Name (none) -> 电压:1kV 电流:1A; Manufacturer (none) -> MDD(辰达半导体); Manufacturer Part (none) -> US1MF; Supplier (none) -> LCSC; Supplier Part (none) -> C64877
- Q1: footprint Package_TO_SOT_SMD:SOT-23 -> easyEDA:SOT-23-3_L2.9-W1.6-P1.90-LS2.8-BR; symbol Transistor_FET:BSS138 -> easyEDA:BSS138-7-F; LCSC Part Name (none) -> 1个N沟道 耐压:50V 电流:200mA; Manufacturer (none) -> DIODES(美台); Manufacturer Part (none) -> BSS138-7-F; Supplier (none) -> LCSC; Supplier Part (none) -> C40912
- R1: value R0Ohm -> 0Ω; footprint (none) -> easyEDA:R1206; symbol Device:R -> easyEDA:1206 J000T5E; LCSC Part Name (none) -> 0Ω ±5% 250mW 厚膜电阻; Manufacturer (none) -> UNI-ROYAL(厚声); Manufacturer Part (none) -> 1206W4J0000T5E; Supplier (none) -> LCSC; Supplier Part (none) -> C19290
- R2, R3, R4: value R10K -> 10kΩ; footprint (none) -> easyEDA:R1206; symbol Device:R -> easyEDA:1206W4F1002T5E; LCSC Part Name (none) -> 10kΩ ±1% 250mW 厚膜电阻; Manufacturer (none) -> UNI-ROYAL(厚声); Manufacturer Part (none) -> 1206W4F1002T5E; Supplier (none) -> LCSC; Supplier Part (none) -> C17902
- R2: renamed from RV2; value R_2.2K -> 2kΩ/2.2K; footprint (none) -> easyEDA:RES-ADJ-TH_3P-L7.1-W6.9-P2.50-L_3362P; symbol Device:R_Potentiometer -> easyEDA:3362P-1-202_C118929; LCSC Part Name (none) -> 2kΩ ±10%; Manufacturer (none) -> BOCHEN(博晨); Manufacturer Part (none) -> 3362P-1-202; Supplier (none) -> LCSC; Supplier Part (none) -> C118929
- R5: value R820 -> 820Ω; footprint (none) -> easyEDA:R1206; symbol Device:R -> easyEDA:1206W4F8200T5E; LCSC Part Name (none) -> 820Ω ±1% 250mW 厚膜电阻; Manufacturer (none) -> UNI-ROYAL(厚声); Manufacturer Part (none) -> 1206W4F8200T5E; Supplier (none) -> LCSC; Supplier Part (none) -> C17984
- RV1: footprint (none) -> easyEDA:RES-ADJ-TH_3362P; symbol Device:R_Potentiometer -> easyEDA:3362P-1-104_C118966; LCSC Part Name (none) -> 100kΩ ±10%; Manufacturer (none) -> BOCHEN(博晨); Manufacturer Part (none) -> 3362P-1-104; Supplier (none) -> LCSC; Supplier Part (none) -> C118966
Connections:
- net +3.3V: now also R3.2; no longer R3.1
- net +5V: now also R2.2, R4.2, U3.8 (VCC+), U7.3; no longer R2.1, R4.1
- net AnalogOut: now also U3.2 (-), U3.6 (-), U3.7
- net DigitalOut: now also R3.1; no longer R3.2
- net GND: now also C1.1, C2.1, RV1.1, U3.4 (GND); no longer C1.2, C2.2, RV1.3
- net at D1.1 (K), RV1.2: now also C2.2, U3.5 (+); no longer C2.1
- net at R2.1: now also R4.1; no longer R4.2
- net at R1.1: now also C1.2, Q1.3 (D), R2.1
- net at R2.2: now also U3.3 (+)
- new net: R14.1, R17.2
- new net: D2.4 (AC), R14.2
- new net: RV1.3, U7.4
- new net: R12.1, U2.2
- new net: R12.2, R13.1
- new net: R17.1, U2.1
- new net: D2.3 (-), U7.1
- new net: D2.1 (+), U7.2
- new net: D2.2 (AC), R13.2
- new net: R1.2, U3.1

Commit message: Feat: Working in PCB files
Parts:
- removed R12, R13, R14: R, symbol Device:R
- added R26, R27, R28: 22K (FHV), ibSolutions:R_Axial_L31.2mm_D1.0mm_P34.0mm_Horizontal, symbol Device:R
- R25: renamed from R17; value R -> 22K (FHV); footprint (none) -> ibSolutions:R_Axial_L31.2mm_D1.0mm_P34.0mm_Horizontal; Comentarios (none) -> Datashee con PEON; Manufacturer (none) -> SHENZHEN JING DA CHENG ELECTRONIC CO., LTD.; Part No (none) -> FVR01B
- U8: renamed from U2; footprint easyEDA:CONN-TH_KF88SA-16.0-2P -> ibSolutions:2Pin_L11.0mm_D1.5mm_P17mm; symbol easyEDA:KF88SA-16.0-2P -> Connector:Conn_01x02_Pin; Comentarios (none) -> Es para soldar directamente el cable; LCSC Part Name 16mm 1x2P 每排P数:2 排数:1 直针 -> (none); Manufacturer KEFA(科发) -> (none); Manufacturer Part KF88SA-16.0-2P -> (none); Supplier LCSC -> (none); Supplier Part C707749 -> (none)
- renumbered C3 to C4, C2 to C5, C1 to C6, D2 to D1, D1 to D2, Q1 to Q4, R4 to R29, R2 to R30, R5 to R31, R1 to R32, R2 to R33, R3 to R34, U3 to U10, U7 to U9
Connections:
- net at R25.2: now also R27.1
- net at D1.4 (AC): now also R27.2
- net at U8.2 (Pin_2): now also R26.1
- net at D1.2 (AC): now also R28.2
- new net: R26.2, R28.1

Commit message: Feat Board Completed, in production
Parts:
- C4, C5: value C -> 100nF; Comments (none) -> -; JLCPCB Part (none) -> C82601; LCSC (none) -> C82601
- C6: Comments (none) -> -; JLCPCB Part (none) -> C24497; LCSC (none) -> C24497
- D1: Comments (none) -> -; JLCPCB Part (none) -> C2983251; LCSC (none) -> C2983251
- D2: value US1MF/1N4007 -> US1MF; Comments (none) -> -; JLCPCB Part (none) -> C64877; LCSC (none) -> C64877
- Q4: value BSS138 -> BSS138-7-F; Comments (none) -> -; JLCPCB Part (none) -> C40912; LCSC (none) -> C40912
- R25, R26, R27, R28: value 22K (FHV) -> R; JLCPCB Part (none) -> -; LCSC (none) -> -; Part No FVR01B -> (none); Supplier (none) -> LCSC; Supplier Part (none) -> -
- R29, R33, R34: Comments (none) -> -; JLCPCB Part (none) -> C17902; LCSC (none) -> C17902
- R30: value 2kΩ/2.2K -> 2kΩ; JLCPCB Part (none) -> C118929; LCSC (none) -> C118929
- R31: JLCPCB Part (none) -> C17984; LCSC (none) -> C17984
- R32: JLCPCB Part (none) -> C19290; LCSC (none) -> C19290
- RV1: value R_100K -> 100kΩ; JLCPCB Part (none) -> C118966; LCSC (none) -> C118966
- U10: value LMV358 -> LMV358IDR; Comments (none) -> -; JLCPCB Part (none) -> C63813; LCSC (none) -> C63813
- U8: value ~ -> Conn_01x02_Pin; JLCPCB Part (none) -> -; LCSC (none) -> -; Supplier (none) -> LCSC; Supplier Part (none) -> -
- U9: value ~ -> Opto Peon; Comentarios (none) -> -; JLCPCB Part (none) -> -; LCSC (none) -> -; Supplier (none) -> PEON; Supplier Part (none) -> -
